File: SPI-I2C-PWM Excersize/PCB/SPI-i2c-PWM --v1.brd (EAGLE design)
At the start: 129.5 x 75.9 mm, 72 parts, among them M1 ARDUINO-DIP28, M1_OSC AS-16.000-18-CRYSTAL

Commit message: updates to i2c-spi scheamtic and board files plus new output images
Parts:
- renumbered M1 to MCU-P1, M1SR to SHIFT_REG_P1, M1_POT to P1_POT, S1 to MCU-C1, S1SR to SHIFT_REG_C1, S1_I2C to C1_I2C, S1_POT to C1_POT, S1_SPI to C1_SPI, S2 to MCU-C2, S2SR to SHIFT_REG_C2, S2_I2C to C2_I2C, S2_POT to C2_POT, S2_PWM to C2_PWM, S2_SPI to C2_SPI, S3 to MCU-C3, S3SR to SHIFT_REG_C3, S3_I2C to C3_I2C, S3_POT to C3_POT, S3_PWM to C3_PWM, S3_SPI to C3_SPI
Connections:
- net M1SR-OE renamed P1-OE
- net M1SR-RCLK renamed P1-RCLK
- net M1SR-SER renamed P1-SER
- net M1SR-SRCLK renamed P1-SRCLK
- net M1SR-SRCLR renamed P1-SRCLR
- net S1SR-OE renamed C1-OE
- net S1SR-RCLK renamed C1-RCLK
- net S1SR-SER renamed C1-SER
- net S1SR-SRCLK renamed C1-SRCLK
- net S1SR-SRCLR renamed C1-SRCLR
- net S1_HELLO_I2C renamed C1_HELLO_I2C
- net S1_HELLO_PWM renamed C1_HELLO_PWM
- net S1_HELLO_SPI renamed C1_HELLO_SPI
- net S2SR-OE renamed C2-OE
- net S2SR-RCLK renamed C2-RCLK
- net S2SR-SER renamed C2-SER
- net S2SR-SRCLK renamed C2-SRCLK
- net S2SR-SRCLR renamed C2-SRCLR
- net S2_HELLO_I2C renamed C2_HELLO_I2C
- net S2_HELLO_PWM renamed C2_HELLO_PWM
- net S2_HELLO_SPI renamed C2_HELLO_SPI
- net S2_ICP1 renamed C2_ICP1
- net S3SR-OE renamed C3-OE
- net S3SR-RCLK renamed C3-RCLK
- net S3SR-SER renamed C3-SER
- net S3SR-SRCLK renamed C3-SRCLK
- net S3SR-SRCLR renamed C3-SRCLR
- net S3_HELLO_I2C renamed C3_HELLO_I2C
- net S3_HELLO_PWM renamed C3_HELLO_PWM
- net S3_HELLO_SPI renamed C3_HELLO_SPI
- net S3_ICP1 renamed C3_ICP1
- net SS1 renamed CS1
- net SS2 renamed CS2
- net SS3 renamed CS3
- removed net M1_POT1: MCU-P1.23, P1_POT.P$2
- removed net S1_POT1: C1_POT.P$2, MCU-C1.26
- removed net S2_POT1: C2_POT.P$2, MCU-C2.26
- removed net S3_POT1: C3_POT.P$2, MCU-C3.26
- new net C1_POT: C1_POT.P$2
- new net C1_POT1: MCU-C1.26
- new net C2_POT: C2_POT.P$2
- new net C2_POT1: MCU-C2.26
- new net C3_POT: C3_POT.P$2
- new net C3_POT1: MCU-C3.26
- new net P1_POT: P1_POT.P$2
- new net P1_POT1: MCU-P1.23
Routing:
- net S3_POT1: track 86.5 -> 0.00 mm
- net C3_POT1: track 0.00 -> 76.4 mm
- net S2_POT1: track 54.9 -> 0.00 mm
- net C2_POT1: track 0.00 -> 54.5 mm
- net S1_POT1: track 51.0 -> 0.00 mm
- net C1_POT1: track 0.00 -> 50.9 mm
- net M1_POT1: track 50.1 -> 0.00 mm
- net P1_POT: track 0.00 -> 49.8 mm
- net CS3: track 23.2 -> 22.0 mm
- net CS2: track 58.3 -> 57.8 mm
