File: SPI-I2C-PWM Excersize/PCB/SPI-i2c-PWM --v1.sch (EAGLE design)
At the start: 72 parts, among them M1 ARDUINO-DIP28, M1_OSC AS-16.000-18-CRYSTAL

Commit message: updates to i2c-spi scheamtic and board files plus new output images
Parts:
- removed M1, S1, S2, S3: ARDUINO-DIP28, peter ford222:ARDUINO-DIP28
- removed M1SR, S1SR, S2SR, S3SR: (no value), pinhead:PINHD-1X8
- removed M1_POT, S1_POT, S2_POT, S3_POT: (no value), peter ford222:POTENTIOMETER-ALLIE
- removed S1_I2C, S2_I2C, S3_I2C: BLUE, led:LEDCHIP-LED0805
- removed S1_SPI, S2_SPI, S3_SPI: GREEN, led:LEDCHIP-LED0805
- removed S2_PWM, S3_PWM: YELLOW, led:LEDCHIP-LED0805
- added C1_I2C, C2_I2C, C3_I2C: BLUE, led:LEDCHIP-LED0805
- added C1_POT, C2_POT, C3_POT, P1_POT: (no value), peter ford222:POTENTIOMETER-ALLIE
- added C1_SPI, C2_SPI, C3_SPI: GREEN, led:LEDCHIP-LED0805
- added C2_PWM, C3_PWM: YELLOW, led:LEDCHIP-LED0805
- added MCU-C1, MCU-C2, MCU-C3, MCU-P1: ARDUINO-DIP28, peter ford222:ARDUINO-DIP28
- added SHIFT_REG_C1, SHIFT_REG_C2, SHIFT_REG_C3, SHIFT_REG_P1: (no value), pinhead:PINHD-1X8
Connections:
- removed net M1SR-OE: M1.PD1(PCINT17/TXD), M1SR.2
- removed net M1SR-RCLK: M1.PD2(PCINT18/INT0), M1SR.3
- removed net M1SR-SER: M1.PD0(PCINT16/RXD), M1SR.1
- removed net M1SR-SRCLK: M1.PD4(PCINT20/XCK/T0), M1SR.4
- removed net M1SR-SRCLR: M1.PD7(PCINT23/AIN1), M1SR.5
- removed net M1_POT1: M1.PC0(ADC0/PCINT8), M1_POT.P$2
- removed net S1SR-OE: S1.PD1(PCINT17/TXD), S1SR.2
- removed net S1SR-RCLK: S1.PD2(PCINT18/INT0), S1SR.3
- removed net S1SR-SER: S1.PD0(PCINT16/RXD), S1SR.1
- removed net S1SR-SRCLK: S1.PD3(PCINT19/OC2B/INT1), S1SR.4
- removed net S1SR-SRCLR: S1.PD4(PCINT20/XCK/T0), S1SR.5
- removed net S1_HELLO_I2C: R9.1, S1.PD6(PCINT22/OC0A/AIN0)
- removed net S1_HELLO_PWM: S1.PD7(PCINT23/AIN1)
- removed net S1_HELLO_SPI: R6.1, S1.PD5(PCINT21/OC0B/T1)
- removed net S1_POT1: S1.PC3(ADC3/PCINT11), S1_POT.P$2
- removed net S2SR-OE: S2.PD1(PCINT17/TXD), S2SR.2
- removed net S2SR-RCLK: S2.PD2(PCINT18/INT0), S2SR.3
- removed net S2SR-SER: S2.PD0(PCINT16/RXD), S2SR.1
- removed net S2SR-SRCLK: S2.PD3(PCINT19/OC2B/INT1), S2SR.4
- removed net S2SR-SRCLR: S2.PD4(PCINT20/XCK/T0), S2SR.5
- removed net S2_HELLO_I2C: R10.1, S2.PD6(PCINT22/OC0A/AIN0)
- removed net S2_HELLO_PWM: R13.1, S2.PD7(PCINT23/AIN1)
- removed net S2_HELLO_SPI: R7.1, S2.PD5(PCINT21/OC0B/T1)
- removed net S2_ICP1: M1.PD5(PCINT21/OC0B/T1), S2.PB0(PCINT0/CLKO/ICP1)
- removed net S2_POT1: S2.PC3(ADC3/PCINT11), S2_POT.P$2
- removed net S3SR-OE: S3.PD1(PCINT17/TXD), S3SR.2
- removed net S3SR-RCLK: S3.PD2(PCINT18/INT0), S3SR.3
- removed net S3SR-SER: S3.PD0(PCINT16/RXD), S3SR.1
- removed net S3SR-SRCLK: S3.PD3(PCINT19/OC2B/INT1), S3SR.4
- removed net S3SR-SRCLR: S3.PD4(PCINT20/XCK/T0), S3SR.5
- removed net S3_HELLO_I2C: R11.1, S3.PD6(PCINT22/OC0A/AIN0)
- removed net S3_HELLO_PWM: R14.1, S3.PD7(PCINT23/AIN1)
- removed net S3_HELLO_SPI: R8.1, S3.PD5(PCINT21/OC0B/T1)
- removed net S3_ICP1: M1.PD6(PCINT22/OC0A/AIN0), S3.PB0(PCINT0/CLKO/ICP1)
- removed net S3_POT1: S3.PC3(ADC3/PCINT11), S3_POT.P$2
- removed net SS1: M1.PB2(SS/OC1B/PCINT2), S1.PB2(SS/OC1B/PCINT2)
- removed net SS2: M1.PB1(OC1A/PCINT1), S2.PB2(SS/OC1B/PCINT2)
- removed net SS3: M1.PB0(PCINT0/CLKO/ICP1), S3.PB2(SS/OC1B/PCINT2)
- new net C1-OE: MCU-C1.PD1(PCINT17/TXD), SHIFT_REG_C1.2
- new net C1-RCLK: MCU-C1.PD2(PCINT18/INT0), SHIFT_REG_C1.3
- new net C1-SER: MCU-C1.PD0(PCINT16/RXD), SHIFT_REG_C1.1
- new net C1-SRCLK: MCU-C1.PD3(PCINT19/OC2B/INT1), SHIFT_REG_C1.4
- new net C1-SRCLR: MCU-C1.PD4(PCINT20/XCK/T0), SHIFT_REG_C1.5
- new net C1_HELLO_I2C: MCU-C1.PD6(PCINT22/OC0A/AIN0), R9.1
- new net C1_HELLO_PWM: MCU-C1.PD7(PCINT23/AIN1)
- new net C1_HELLO_SPI: MCU-C1.PD5(PCINT21/OC0B/T1), R6.1
- new net C1_POT: C1_POT.P$2
- new net C1_POT1: MCU-C1.PC3(ADC3/PCINT11)
- new net C2-OE: MCU-C2.PD1(PCINT17/TXD), SHIFT_REG_C2.2
- new net C2-RCLK: MCU-C2.PD2(PCINT18/INT0), SHIFT_REG_C2.3
- new net C2-SER: MCU-C2.PD0(PCINT16/RXD), SHIFT_REG_C2.1
- new net C2-SRCLK: MCU-C2.PD3(PCINT19/OC2B/INT1), SHIFT_REG_C2.4
- new net C2-SRCLR: MCU-C2.PD4(PCINT20/XCK/T0), SHIFT_REG_C2.5
- new net C2_HELLO_I2C: MCU-C2.PD6(PCINT22/OC0A/AIN0), R10.1
- new net C2_HELLO_PWM: MCU-C2.PD7(PCINT23/AIN1), R13.1
- new net C2_HELLO_SPI: MCU-C2.PD5(PCINT21/OC0B/T1), R7.1
- new net C2_ICP1: MCU-C2.PB0(PCINT0/CLKO/ICP1), MCU-P1.PD5(PCINT21/OC0B/T1)
- new net C2_POT: C2_POT.P$2
- new net C2_POT1: MCU-C2.PC3(ADC3/PCINT11)
- new net C3-OE: MCU-C3.PD1(PCINT17/TXD), SHIFT_REG_C3.2
- new net C3-RCLK: MCU-C3.PD2(PCINT18/INT0), SHIFT_REG_C3.3
- new net C3-SER: MCU-C3.PD0(PCINT16/RXD), SHIFT_REG_C3.1
- new net C3-SRCLK: MCU-C3.PD3(PCINT19/OC2B/INT1), SHIFT_REG_C3.4
- new net C3-SRCLR: MCU-C3.PD4(PCINT20/XCK/T0), SHIFT_REG_C3.5
- new net C3_HELLO_I2C: MCU-C3.PD6(PCINT22/OC0A/AIN0), R11.1
- new net C3_HELLO_PWM: MCU-C3.PD7(PCINT23/AIN1), R14.1
- new net C3_HELLO_SPI: MCU-C3.PD5(PCINT21/OC0B/T1), R8.1
- new net C3_ICP1: MCU-C3.PB0(PCINT0/CLKO/ICP1), MCU-P1.PD6(PCINT22/OC0A/AIN0)
- new net C3_POT: C3_POT.P$2
- new net C3_POT1: MCU-C3.PC3(ADC3/PCINT11)
- new net CS1: MCU-C1.PB2(SS/OC1B/PCINT2), MCU-P1.PB2(SS/OC1B/PCINT2)
- new net CS2: MCU-C2.PB2(SS/OC1B/PCINT2), MCU-P1.PB1(OC1A/PCINT1)
- new net CS3: MCU-C3.PB2(SS/OC1B/PCINT2), MCU-P1.PB0(PCINT0/CLKO/ICP1)
- new net P1-OE: MCU-P1.PD1(PCINT17/TXD), SHIFT_REG_P1.2
- new net P1-RCLK: MCU-P1.PD2(PCINT18/INT0), SHIFT_REG_P1.3
- new net P1-SER: MCU-P1.PD0(PCINT16/RXD), SHIFT_REG_P1.1
- new net P1-SRCLK: MCU-P1.PD4(PCINT20/XCK/T0), SHIFT_REG_P1.4
- new net P1-SRCLR: MCU-P1.PD7(PCINT23/AIN1), SHIFT_REG_P1.5
- new net P1_POT: P1_POT.P$2
- new net P1_POT1: MCU-P1.PC0(ADC0/PCINT8)
- net 8B_INPUT_LADDER: now also MCU-P1.PC3(ADC3/PCINT11); no longer M1.PC3(ADC3/PCINT11)
- net CHIP_SELECT_LADDER: now also MCU-P1.PC1(ADC1/PCINT9); no longer M1.PC1(ADC1/PCINT9)
- net COM_SELECT_LADDER: now also MCU-P1.PC2(ADC2/PCINT10); no longer M1.PC2(ADC2/PCINT10)
- net GND: now also C1_I2C.C, C1_POT.P$3, C1_SPI.C, C2_I2C.C, C2_POT.P$3, C2_PWM.C, C2_SPI.C, C3_I2C.C, C3_POT.P$3, C3_PWM.C, C3_SPI.C, MCU-C1.GND, MCU-C1.GND2, MCU-C2.GND, MCU-C2.GND2, MCU-C3.GND, MCU-C3.GND2, MCU-P1.GND, MCU-P1.GND2, P1_POT.P$3, SHIFT_REG_C1.8, SHIFT_REG_C2.8, SHIFT_REG_C3.8, SHIFT_REG_P1.8; no longer M1.GND, M1.GND2, M1SR.8, M1_POT.P$3, S1.GND, S1.GND2, S1SR.8, S1_I2C.C, S1_POT.P$3, S1_SPI.C, S2.GND, S2.GND2, S2SR.8, S2_I2C.C, S2_POT.P$3, S2_PWM.C, S2_SPI.C, S3.GND, S3.GND2, S3SR.8, S3_I2C.C, S3_POT.P$3, S3_PWM.C, S3_SPI.C
- net MISO: now also MCU-C1.PB4(MISO/PCINT4), MCU-C2.PB4(MISO/PCINT4), MCU-C3.PB4(MISO/PCINT4), MCU-P1.PB4(MISO/PCINT4); no longer M1.PB4(MISO/PCINT4), S1.PB4(MISO/PCINT4), S2.PB4(MISO/PCINT4), S3.PB4(MISO/PCINT4)
- net MOSI: now also MCU-C1.PB3(MOSI/OC2A/PCINT3), MCU-C2.PB3(MOSI/OC2A/PCINT3), MCU-C3.PB3(MOSI/OC2A/PCINT3), MCU-P1.PB3(MOSI/OC2A/PCINT3); no longer M1.PB3(MOSI/OC2A/PCINT3), S1.PB3(MOSI/OC2A/PCINT3), S2.PB3(MOSI/OC2A/PCINT3), S3.PB3(MOSI/OC2A/PCINT3)
- net N$10: now also MCU-C3.PB7(PCINT7/XTAL2/TOSC2); no longer S3.PB7(PCINT7/XTAL2/TOSC2)
- net N$12: now also C1_SPI.A; no longer S1_SPI.A
- net N$13: now also C2_SPI.A; no longer S2_SPI.A
- net N$14: now also C3_SPI.A; no longer S3_SPI.A
- net N$15: now also C1_I2C.A; no longer S1_I2C.A
- net N$16: now also C2_I2C.A; no longer S2_I2C.A
- net N$17: now also C3_I2C.A; no longer S3_I2C.A
- net N$19: now also C2_PWM.A; no longer S2_PWM.A
- net N$2: now also MCU-C1.PB6(PCINT6/XTAL1/TOSC1); no longer S1.PB6(PCINT6/XTAL1/TOSC1)
- net N$20: now also C3_PWM.A; no longer S3_PWM.A
- net N$3: now also MCU-C1.PB7(PCINT7/XTAL2/TOSC2); no longer S1.PB7(PCINT7/XTAL2/TOSC2)
- net N$5: now also MCU-P1.PB6(PCINT6/XTAL1/TOSC1); no longer M1.PB6(PCINT6/XTAL1/TOSC1)
- net N$6: now also MCU-P1.PB7(PCINT7/XTAL2/TOSC2); no longer M1.PB7(PCINT7/XTAL2/TOSC2)
- net N$7: now also MCU-C2.PB6(PCINT6/XTAL1/TOSC1); no longer S2.PB6(PCINT6/XTAL1/TOSC1)
- net N$8: now also MCU-C2.PB7(PCINT7/XTAL2/TOSC2); no longer S2.PB7(PCINT7/XTAL2/TOSC2)
- net N$9: now also MCU-C3.PB6(PCINT6/XTAL1/TOSC1); no longer S3.PB6(PCINT6/XTAL1/TOSC1)
- net RESET1: now also MCU-C1.PC6(PCINT14/RESET); no longer S1.PC6(PCINT14/RESET)
- net RESET2: now also MCU-C2.PC6(PCINT14/RESET); no longer S2.PC6(PCINT14/RESET)
- net RESET3: now also MCU-C3.PC6(PCINT14/RESET); no longer S3.PC6(PCINT14/RESET)
- net RESET_BUTTON: now also MCU-P1.PC6(PCINT14/RESET); no longer M1.PC6(PCINT14/RESET)
- net SCK: now also MCU-C1.PB5(SCK/PCINT5), MCU-C2.PB5(SCK/PCINT5), MCU-C3.PB5(SCK/PCINT5), MCU-P1.PB5(SCK/PCINT5); no longer M1.PB5(SCK/PCINT5), S1.PB5(SCK/PCINT5), S2.PB5(SCK/PCINT5), S3.PB5(SCK/PCINT5)
- net SCL: now also MCU-C1.PC5(ADC5/SCL/PCINT13), MCU-C2.PC5(ADC5/SCL/PCINT13), MCU-C3.PC5(ADC5/SCL/PCINT13), MCU-P1.PC5(ADC5/SCL/PCINT13); no longer M1.PC5(ADC5/SCL/PCINT13), S1.PC5(ADC5/SCL/PCINT13), S2.PC5(ADC5/SCL/PCINT13), S3.PC5(ADC5/SCL/PCINT13)
- net SDA: now also MCU-C1.PC4(ADC4/SDA/PCINT12), MCU-C2.PC4(ADC4/SDA/PCINT12), MCU-C3.PC4(ADC4/SDA/PCINT12), MCU-P1.PC4(ADC4/SDA/PCINT12); no longer M1.PC4(ADC4/SDA/PCINT12), S1.PC4(ADC4/SDA/PCINT12), S2.PC4(ADC4/SDA/PCINT12), S3.PC4(ADC4/SDA/PCINT12)
- net TRANSMIT_BUTTON: now also MCU-P1.PD3(PCINT19/OC2B/INT1); no longer M1.PD3(PCINT19/OC2B/INT1)
- net VCC_ARDUINO: now also C1_POT.P$1, C2_POT.P$1, C3_POT.P$1, MCU-C1.AREF, MCU-C1.AVCC, MCU-C1.VCC, MCU-C2.AREF, MCU-C2.AVCC, MCU-C2.VCC, MCU-C3.AREF, MCU-C3.AVCC, MCU-C3.VCC, MCU-P1.AREF, MCU-P1.AVCC, MCU-P1.VCC, P1_POT.P$1, SHIFT_REG_C1.7, SHIFT_REG_C2.7, SHIFT_REG_C3.7, SHIFT_REG_P1.7; no longer M1.AREF, M1.AVCC, M1.VCC, M1SR.7, M1_POT.P$1, S1.AREF, S1.AVCC, S1.VCC, S1SR.7, S1_POT.P$1, S2.AREF, S2.AVCC, S2.VCC, S2SR.7, S2_POT.P$1, S3.AREF, S3.AVCC, S3.VCC, S3SR.7, S3_POT.P$1
Other:
- note added: "C1 Peripherals"
- note added: "C2 Peripherals"
- note added: "C3 Peripherals"
- note added: "CHILDREN"
- note added: "P1 Peripherals"
- note added: "PARENT"
- moved on the sheet: 8B_INPUT_DIP, 8B_INPUT_R2R, C1, C10, C11, C12, C13, C14, C15, C16, C17, C18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
